Commit message: fix: lidar self-collision causing false stop; disable ray visualization

File: ros2_ws/src/mower_description/urdf/mower.urdf.xacro (robot description, xacro)
@@ -67,7 +67,4 @@
       <material name="grey"><color rgba="0.3 0.3 0.3 1"/></material>
     </visual>
-    <collision>
-      <geometry><cylinder radius="0.035" length="0.04"/></geometry>
-    </collision>
     <inertial>
       <mass value="0.15"/>
@@ -107,5 +104,5 @@
     <sensor name="lidar" type="ray">
       <pose>0 0 0 0 0 0</pose>
-      <visualize>true</visualize>
+      <visualize>false</visualize>
       <update_rate>10</update_rate>
       <ray>

Commit message: fix: move lidar ahead of chassis front edge to stop front self-hit

File: ros2_ws/src/mower_description/urdf/mower.urdf.xacro (robot description, xacro)
@@ -75,5 +75,5 @@
     <parent link="base_link"/>
     <child link="lidar_link"/>
-    <origin xyz="${chassis_length/2 - 0.05} 0 ${chassis_height/2 + 0.02}" rpy="0 0 0"/>
+    <origin xyz="${chassis_length/2 + 0.02} 0 ${chassis_height/2 + 0.02}" rpy="0 0 0"/>
   </joint>
   <gazebo reference="caster_link">
